Commit message: Added collision meshes.

File: robots/LRMate200iD_description.URDF (robot description, URDF)
Before this commit: robot LRMate200iD_description, 7 links, 6 joints
Links:
- link base_link: geometry collision mesh filename=package://LRMate200iD_description/meshes/base_link_collisio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; visual mesh filename=package://LRMate200iD_description/meshes/base_link.STL
- link bicep: geometry collision mesh filename=package://LRMate200iD_description/meshes/bicep_collision.STL; visual mesh filename=package://LRMate200iD_description/meshes/bicep.STL
- link elbow: geometry collision mesh filename=package://LRMate200iD_description/meshes/elbow_collision.STL; visual mesh filename=package://LRMate200iD_description/meshes/elbow.STL
- link forearm: geometry collision mesh filename=package://LRMate200iD_description/meshes/forearm_collision.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; visual mesh filename=package://LRMate200iD_description/meshes/forearm.STL
- link palm: geometry collision mesh filename=package://LRMate200iD_description/meshes/palm_collision.STL; visual mesh filename=package://LRMate200iD_description/meshes/palm.STL
- link shoulder: geometry collision mesh filename=package://LRMate200iD_description/meshes/shoulder_collision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; visual mesh filename=package://LRMate200iD_description/meshes/shoulder.STL
- link wrist: geometry collision mesh filename=package://LRMate200iD_description/meshes/wrist_collision.STL; visual mesh filename=package://LRMate200iD_description/meshes/wrist.STL

Commit message: Removed inertia tag from base link.

File: robots/LRMate200iD_description.URDF (robot description, URDF)
Before this commit: robot LRMate200iD_description, 7 links, 6 joints
Links:
- link base_link: mass 4.85330591768461E-10 -> None

Commit message: Revised inertial properties

File: robots/LRMate200iD_description.URDF (robot description, URDF)
Before this commit: robot LRMate200iD_description, 7 links, 6 joints
Links:
- link base_link: mass None -> 6.28702953522501
- link bicep: mass 6.3617E-10 -> 8.24093772313152
- link elbow: mass 2.4013E-10 -> 3.11070759102685
- link forearm: mass 2.0398E-10 -> 2.64233524900363
- link palm: mass 1.33888429975585E-12 -> 0.017344
- link shoulder: mass 3.1897E-10 -> 4.13202512738557
- link wrist: mass 4.32840002975359E-11 -> 0.560705873959261

Commit message: Updated velocity and torque limits; added transmission file.

File: robots/LRMate200iD_description.URDF (robot description, URDF)
Before this commit: robot LRMate200iD_description, 7 links, 6 joints
Joints:
- joint elbow_pitch: limit lower=-3.577924967 upper=1.204277184 effort=0 velocity=0 -> lower=-3.577924967 upper=1.204277184 effort=308 velocity=9.075716
- joint elbow_roll: limit lower=-3.316125579 upper=3.316125579 effort=0 velocity=0 -> lower=-3.316125579 upper=3.316125579 effort=20 velocity=9.773848
- joint shoulder_pitch: limit lower=-1.919862177 upper=2.094395102 effort=0 velocity=0 -> lower=-1.919862177 upper=2.094395102 effort=308 velocity=8.028518
- joint shoulder_yaw: limit lower=-2.967059728 upper=2.967059728 effort=0 velocity=0 -> lower=-2.967059728 upper=2.967059728 effort=135 velocity=8.028518
- joint wrist_pitch: limit lower=-2.094395102 upper=2.094395102 effort=0 velocity=0 -> lower=-2.094395102 upper=2.094395102 effort=20 velocity=9.773848
- joint wrist_roll: limit lower=-6.283185307 upper=6.283185307 effort=0 velocity=0 -> lower=-6.283185307 upper=6.283185307 effort=10 velocity=15.70797
