Commit message: Fixed name and added launchfile tests.

File: robots/lrmate_200id_description.URDF (robot description, URDF)
Before this commit: robot LRMate200iD_description, 7 links, 6 joints
Links:
- link base_link: geometry collision mesh filename=package://lrmate_200id_description/meshes/base_link_collisi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; visual mesh filename=package://lrmate_200id_description/meshes/base_link.STL
- link bicep: geometry collision mesh filename=package://lrmate_200id_description/meshes/bicep_collision.S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; visual mesh filename=package://lrmate_200id_description/meshes/bicep.STL
- link elbow: geometry collision mesh filename=package://lrmate_200id_description/meshes/elbow_collision.S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; visual mesh filename=package://lrmate_200id_description/meshes/elbow.STL
- link forearm: geometry collision mesh filename=package://lrmate_200id_description/meshes/forearm_collision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; visual mesh filename=package://lrmate_200id_description/meshes/forearm.STL
- link palm: geometry collision mesh filename=package://lrmate_200id_description/meshes/palm_collision.STL; visual mesh filename=package://lrmate_200id_description/meshes/palm.STL
- link shoulder: geometry collision mesh filename=package://lrmate_200id_description/meshes/shoulder_collisio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; visual mesh filename=package://lrmate_200id_description/meshes/shoulder.STL
- link wrist: geometry collision mesh filename=package://lrmate_200id_description/meshes/wrist_collision.S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; visual mesh filename=package://lrmate_200id_description/meshes/wrist.STL
